Commit message: fix: code cleanup

File: rover_description/urdf/bot/bot.xacro (robot description, xacro)
@@ -1,7 +1,8 @@
 <?xml version="1.0" ?>
+<!-- working_file -->
 <robot name="savvyage" xmlns:xacro="http://www.ros.org/wiki/xacro" >
-  <xacro:include filename="$(find bot_description)/urdf/materials.xacro" />
-  <xacro:include filename="$(find bot_description)/urdf/bot.gazebo" />
-  <xacro:include filename="$(find bot_description)/urdf/macros.xacro" />
+  <xacro:include filename="$(find rover_description)/urdf/materials.xacro" />
+  <xacro:include filename="$(find rover_description)/urdf/bot/bot.gazebo" />
+  <xacro:include filename="$(find rover_description)/urdf/bot/macros.xacro" />
   <xacro:property name="camera_link" value="0.08" /> <!-- Size of square 'camera' box -->
   <link name="link_chassis">

File: rover_description/urdf/bot/bot2.xacro (robot description, xacro)
@@ -1,7 +1,8 @@
 <?xml version="1.0" ?>
+<!-- working fle -->
 <robot name="savvyage" xmlns:xacro="http://www.ros.org/wiki/xacro" >
-  <xacro:include filename="$(find bot_description)/urdf/materials.xacro" />
-  <xacro:include filename="$(find bot_description)/urdf/bot.gazebo" />
-  <xacro:include filename="$(find bot_description)/urdf/macros.xacro" />
+  <xacro:include filename="$(find rover_description)/urdf/materials.xacro" />
+  <xacro:include filename="$(find rover_description)/urdf/bot/bot.gazebo" />
+  <xacro:include filename="$(find rover_description)/urdf/bot/macros.xacro" />
   <xacro:property name="camera_link" value="0.08" /> <!-- Size of square 'camera' box -->
   <xacro:property name="scale" value="2" />

File: rover_description/urdf/bot/macros.xacro (robot description, xacro)
@@ -1,3 +1,4 @@
 <?xml version="1.0"?>
+<!-- used inside bot -->
 <robot xmlns:xacro="http://www.ros.org/wiki/xacro">
     <xacro:macro name="link_wheel" params="name">

File: rover_description/urdf/materials.xacro (robot description, xacro)
@@ -1,3 +1,2 @@
-// No changes were made
 <?xml version="1.0" ?>
 <robot>

File: rover_description/urdf/rover/rover.urdf (robot description, URDF)
Before this commit: robot rover, 31 links, 30 joints
Links:
- link Left_bogie: geometry collision mesh filename=package://rover_description/meshes/Left_bogie.STL; visual mesh filename=package://rover_description/meshes/Left_bogie.STL
- link Left_rocker: geometry collision mesh filename=package://rover_description/meshes/Left_rocker.STL; visual mesh filename=package://rover_description/meshes/Left_rocker.STL
- link Right_bogie: geometry collision mesh filename=package://rover_description/meshes/Right_bogie.STL; visual mesh filename=package://rover_description/meshes/Right_bogie.STL
- link Right_rocker: geometry collision mesh filename=package://rover_description/meshes/Right_rocker.STL; visual mesh filename=package://rover_description/meshes/Right_rocker.STL
- link ball-left-down: geometry collision mesh filename=package://rover_description/meshes/ball-left-down.STL; visual mesh filename=package://rover_description/meshes/ball-left-down.STL
- link ball-right-down: geometry collision mesh filename=package://rover_description/meshes/ball-right-down.STL; visual mesh filename=package://rover_description/meshes/ball-right-down.STL
- link base_link: geometry collision mesh filename=package://rover_description/meshes/base_link.STL; visual mesh filename=package://rover_description/meshes/base_link.STL
- link connector-link-1: geometry collision mesh filename=package://rover_description/meshes/connector-link-1.STL; visual mesh filename=package://rover_description/meshes/connector-link-1.STL
- link connector-link-2: geometry collision mesh filename=package://rover_description/meshes/connector-link-2.STL; visual mesh filename=package://rover_description/meshes/connector-link-2.STL
- link left-rod: geometry collision mesh filename=package://rover_description/meshes/left-rod.STL; visual mesh filename=package://rover_description/meshes/left-rod.STL
- link right-rod: geometry collision mesh filename=package://rover_description/meshes/right-rod.STL; visual mesh filename=package://rover_description/meshes/right-rod.STL
- link socket-left: geometry collision mesh filename=package://rover_description/meshes/socket-left.STL; visual mesh filename=package://rover_description/meshes/socket-left.STL
- link socket-left-down: geometry collision mesh filename=package://rover_description/meshes/socket-left-down.STL; visual mesh filename=package://rover_description/meshes/socket-left-down.STL
- link socket-right: geometry collision mesh filename=package://rover_description/meshes/socket-right.STL; visual mesh filename=package://rover_description/meshes/socket-right.STL
- link socket-right-down: geometry collision mesh filename=package://rover_description/meshes/socket-right-down.STL; visual mesh filename=package://rover_description/meshes/socket-right-down.STL
- link triangle-ball-left: geometry collision mesh filename=package://rover_description/meshes/triangle-ball-left.STL; visual mesh filename=package://rover_description/meshes/triangle-ball-left.STL
- link triangle-ball-right: geometry collision mesh filename=package://rover_description/meshes/triangle-ball-right.STL; visual mesh filename=package://rover_description/meshes/triangle-ball-right.STL
- link triangle-connector: geometry collision mesh filename=package://rover_description/meshes/triangle-connector-l.STL; visual mesh filename=package://rover_description/meshes/triangle-connector-l.STL
- link triangle-left: geometry collision mesh filename=package://rover_description/meshes/triangle-left.STL; visual mesh filename=package://rover_description/meshes/triangle-left.STL
- link triangle-right: geometry collision mesh filename=package://rover_description/meshes/triangle-right.STL; visual mesh filename=package://rover_description/meshes/triangle-right.STL
- link wheel_1: geometry collision mesh filename=package://rover_description/meshes/wheel_1.STL; visual mesh filename=package://rover_description/meshes/wheel_1.STL
- link wheel_2: geometry collision mesh filename=package://rover_description/meshes/wheel_2.STL; visual mesh filename=package://rover_description/meshes/wheel_2.STL
- link wheel_3: geometry collision mesh filename=package://rover_description/meshes/wheel_3.STL; visual mesh filename=package://rover_description/meshes/wheel_3.STL
- link wheel_4: geometry collision mesh filename=package://rover_description/meshes/wheel_4.STL; visual mesh filename=package://rover_description/meshes/wheel_4.STL
- link wheel_5: geometry collision mesh filename=package://rover_description/meshes/wheel_5.STL; visual mesh filename=package://rover_description/meshes/wheel_5.STL
- link wheel_6: geometry collision mesh filename=package://rover_description/meshes/wheel_5.STL; visual mesh filename=package://rover_description/meshes/wheel_5.STL
