Commit message: feat: added rover_gazebosim

File: rover_description/urdf/rover/rover.urdf (robot description, URDF)
Before this commit: robot rover, 31 links, 30 joints
Links:
- link Left_bogie: geometry collision mesh filename=$(find rover_description)/meshes/Left_bogie.STL; visual mesh filename=$(find rover_description)/meshes/Left_bogie.STL
- link Left_rocker: geometry collision mesh filename=$(find rover_description)/meshes/Left_rocker.STL; visual mesh filename=$(find rover_description)/meshes/Left_rocker.STL
- link Right_bogie: geometry collision mesh filename=$(find rover_description)/meshes/Right_bogie.STL; visual mesh filename=$(find rover_description)/meshes/Right_bogie.STL
- link Right_rocker: geometry collision mesh filename=$(find rover_description)/meshes/Right_rocker.STL; visual mesh filename=$(find rover_description)/meshes/Right_rocker.STL
- link ball-left-down: geometry collision mesh filename=$(find rover_description)/meshes/ball-left-down.STL; visual mesh filename=$(find rover_description)/meshes/ball-left-down.STL
- link ball-right-down: geometry collision mesh filename=$(find rover_description)/meshes/ball-right-down.STL; visual mesh filename=$(find rover_description)/meshes/ball-right-down.STL
- link base_link: geometry collision mesh filename=$(find rover_description)/meshes/base_link.STL; visual mesh filename=$(find rover_description)/meshes/base_link.STL
- link connector-link-1: geometry collision mesh filename=$(find rover_description)/meshes/connector-link-1.STL; visual mesh filename=$(find rover_description)/meshes/connector-link-1.STL
- link connector-link-2: geometry collision mesh filename=$(find rover_description)/meshes/connector-link-2.STL; visual mesh filename=$(find rover_description)/meshes/connector-link-2.STL
- link left-rod: geometry collision mesh filename=$(find rover_description)/meshes/left-rod.STL; visual mesh filename=$(find rover_description)/meshes/left-rod.STL
- link right-rod: geometry collision mesh filename=$(find rover_description)/meshes/right-rod.STL; visual mesh filename=$(find rover_description)/meshes/right-rod.STL
- link socket-left: geometry collision mesh filename=$(find rover_description)/meshes/socket-left.STL; visual mesh filename=$(find rover_description)/meshes/socket-left.STL
- link socket-left-down: geometry collision mesh filename=$(find rover_description)/meshes/socket-left-down.STL; visual mesh filename=$(find rover_description)/meshes/socket-left-down.STL
- link socket-right: geometry collision mesh filename=$(find rover_description)/meshes/socket-right.STL; visual mesh filename=$(find rover_description)/meshes/socket-right.STL
- link socket-right-down: geometry collision mesh filename=$(find rover_description)/meshes/socket-right-down.STL; visual mesh filename=$(find rover_description)/meshes/socket-right-down.STL
- link triangle-ball-left: geometry collision mesh filename=$(find rover_description)/meshes/triangle-ball-left.STL; visual mesh filename=$(find rover_description)/meshes/triangle-ball-left.STL
- link triangle-ball-right: geometry collision mesh filename=$(find rover_description)/meshes/triangle-ball-right.STL; visual mesh filename=$(find rover_description)/meshes/triangle-ball-right.STL
- link triangle-connector: geometry collision mesh filename=$(find rover_description)/meshes/triangle-connector-l.STL; visual mesh filename=$(find rover_description)/meshes/triangle-connector-l.STL
- link triangle-left: geometry collision mesh filename=$(find rover_description)/meshes/triangle-left.STL; visual mesh filename=$(find rover_description)/meshes/triangle-left.STL
- link triangle-right: geometry collision mesh filename=$(find rover_description)/meshes/triangle-right.STL; visual mesh filename=$(find rover_description)/meshes/triangle-right.STL
- link wheel_1: geometry collision mesh filename=$(find rover_description)/meshes/wheel_1.STL; visual mesh filename=$(find rover_description)/meshes/wheel_1.STL
- link wheel_2: geometry collision mesh filename=$(find rover_description)/meshes/wheel_2.STL; visual mesh filename=$(find rover_description)/meshes/wheel_2.STL
- link wheel_3: geometry collision mesh filename=$(find rover_description)/meshes/wheel_3.STL; visual mesh filename=$(find rover_description)/meshes/wheel_3.STL
- link wheel_4: geometry collision mesh filename=$(find rover_description)/meshes/wheel_4.STL; visual mesh filename=$(find rover_description)/meshes/wheel_4.STL
- link wheel_5: geometry collision mesh filename=$(find rover_description)/meshes/wheel_5.STL; visual mesh filename=$(find rover_description)/meshes/wheel_5.STL
- link wheel_6: geometry collision mesh filename=$(find rover_description)/meshes/wheel_5.STL; visual mesh filename=$(find rover_description)/meshes/wheel_5.STL
Joints:
- joint ball-socket-left: type floating -> fixed
- joint ball-socket-right: type floating -> fixed
- joint joint1: type continuous -> fixed
- joint joint2: type continuous -> fixed
- joint s-joint-left: type revolute -> fixed
- joint s-joint-left-down: type revolute -> fixed
- joint s-joint-right: type revolute -> fixed

Commit message: feat: added new packages

File: rover_description/urdf/rover/rover.urdf (robot description, URDF)
Before this commit: robot rover, 31 links, 30 joints
Links:
- removed link mrt/camera_link
- added link camera_link, mass 1e-5; collision cylinder length=0.005 radius=0.005; visual cylinder length=0.005 radius=0.005
Joints:
- joint camera_joint: child mrt/camera_link -> camera_link; type continuous -> fixed
- joint camera_optical_joint: parent mrt/camera_link -> camera_link
